Commit message: .

File: robots/pioneer3at.xacro (robot description, xacro)
@@ -397,23 +397,69 @@
     </joint>
   <gazebo reference="p3at_back_${suffix}_wheel">
-    <kp>1000000.0</kp> <!-- kp and kd for rubber -->
-    <kd>100.0</kd>
+    <kp>100000000000000000000000000000000000000000000000.0</kp> <!-- kp and kd for rubber -->
+    <kd>1.0</kd>
     <mu1>1.0</mu1>
     <mu2>1.0</mu2>
-    <fdir1>1 0 0</fdir1> <!-- is this correct? -->
-    <maxVel>1.0</maxVel>
+    <fdir1>0 0 0</fdir1> <!-- is this correct? -->
+    <maxVel>2.0</maxVel>
     <minDepth>0.00</minDepth>
   </gazebo>
   <gazebo reference="p3at_front_${suffix}_wheel">
-    <kp>1000000.0</kp> <!-- kp and kd for rubber -->
-    <kd>100.0</kd>
+    <kp>100000000000000000000000000000000000000000000000.0</kp> <!-- kp and kd for rubber -->
+    <kd>1.0</kd>
     <mu1>1.0</mu1>
     <mu2>1.0</mu2>
-    <fdir1>1 0 0</fdir1> <!-- is this correct? -->
-    <maxVel>1.0</maxVel>
+    <fdir1>0 0 0</fdir1> <!-- is this correct? -->
+    <maxVel>2.0</maxVel>
     <minDepth>0.00</minDepth>
   </gazebo>
+  <transmission name="tran_p3at_front_left_wheel_joint">
+    <type>transmission_interface/SimpleTransmission</type>
+    <joint name="p3at_front_left_wheel_joint">
+      <hardwareInterface>hardware_interface/EffortJointInterface</hardwareInterface>
+    </joint>
+    <actuator name="motor_p3at_front_left_wheel_joint">
+      <hardwareInterface>hardware_interface/EffortJointInterface</hardwareInterface>
+      <mechanicalReduction>1</mechanicalReduction>
+    </actuator>
+  </transmission>
+    <transmission name="tran_p3at_front_right_wheel_joint">
+    <type>transmission_interface/SimpleTransmission</type>
+    <joint name="p3at_front_right_wheel_joint">
+      <hardwareInterface>hardware_interface/EffortJointInterface</hardwareInterface>
+    </joint>
+    <actuator name="motor_p3at_front_right_wheel_joint">
+      <hardwareInterface>hardware_interface/EffortJointInterface</hardwareInterface>
+      <mechanicalReduction>1</mechanicalReduction>
+    </actuator>
+  </transmission>
+    <transmission name="tran_p3at_back_left_wheel_joint">
+    <type>transmission_interface/SimpleTransmission</type>
+    <joint name="p3at_back_left_wheel_joint">
+      <hardwareInterface>hardware_interface/EffortJointInterface</hardwareInterface>
+    </joint>
+    <actuator name="motor_p3at_back_left_wheel_joint">
+      <hardwareInterface>hardware_interface/EffortJointInterface</hardwareInterface>
+      <mechanicalReduction>1</mechanicalReduction>
+    </actuator>
+  </transmission>
+    <transmission name="tran_p3at_back_right_wheel_joint">
+    <type>transmission_interface/SimpleTransmission</type>
+    <joint name="p3at_back_right_wheel_joint">
+      <hardwareInterface>hardware_interface/EffortJointInterface</hardwareInterface>
+    </joint>
+    <actuator name="motor_p3at_back_right_wheel_joint">
+      <hardwareInterface>hardware_interface/EffortJointInterface</hardwareInterface>
+      <mechanicalReduction>1</mechanicalReduction>
+    </actuator>
+  </transmission>
 </xacro:macro>
 <xacro:macro name="p3at_gazebo_ext">
+   <gazebo>
+    <plugin name="gazebo_ros_control" filename="libgazebo_ros_control.so">
+      <robotSimType>gazebo_ros_control/DefaultRobotHWSim</robotSimType>
+      <robotNamespace>/pioneer3at</robotNamespace>
+    </plugin>
+  </gazebo>
 <gazebo>
   <plugin name="skid_steer_drive_controller" filename="libgazebo_ros_skid_steer_drive.so">
